File: AP.kicad_sch (KiCad schematic)
At the start: 21 parts

Commit message: Added Custom Lib
Parts:
- added D?: LED_YawDamping, symbol Device:LED
- added D?: LED_HeadingMode, symbol Device:LED
- added D?: LED_FlightDirector, symbol Device:LED
- added D?: LED_NavMode, symbol Device:LED
- added D?: LED_RollHold, symbol Device:LED
- added D?: LED_VSHold, symbol Device:LED
- added D?: LED_ApproachMode, symbol Device:LED
- added D?: LED_IASHold, symbol Device:LED
- added D?: LED_AP, symbol Device:LED
- added D?: LED_AltHold, symbol Device:LED
- added D?: LED_VNAV, symbol Device:LED
- added D?: LED_PitchHold, symbol Device:LED
- added U?: MAX6971ANG, Package_DIP:DIP-24_W7.62mm_Socket, symbol LibForAP:MAX6971ANG
Connections:
- net VCC: now also D?.2 (A), D?.2 (A), D?.2 (A), D?.2 (A), D?.2 (A), D?.2 (A), D?.2 (A), D?.2 (A), D?.2 (A), D?.2 (A), D?.2 (A), D?.2 (A)
- net LED_DataLatch: now reaches U?.33 (RB0/AN12/INT0/FLT0/SDI/SDA)
- net LED_DIN: now reaches U?.34 (RB1/AN10/INT1/SCK/SCL)
- net LED_CLK: now reaches U?.35 (RB2/AN8/INT2/VMO)
- net LED_lowEN: now reaches U?.36 (RB3/AN9/CCP2/VPO)

Commit message: Save from Work
Parts:
- added R?: 320 Ohms, symbol Device:R
Connections:
- net GND: now also U?.1 (GND), R?.2
- net LED_CLK: now also U?.3 (CLK)
- net LED_DIN: now also U?.2 (DIN)
- net LED_DataLatch: now also U?.4 (LE)
- net LED_lowEN: now also U?.21 (OE_low)
- net VCC: now also U?.24 (V+)
- net at D?.1 (K): now also U?.12 (OUT7)
- net at D?.1 (K): now also U?.7 (OUT2)
- net at D?.1 (K): now also U?.11 (OUT6)
- net at U?.10 (OUT5): now also D?.1 (K)
- net at U?.13 (OUT8): now also D?.1 (K)
- net at U?.14 (OUT9): now also D?.1 (K)
- net at U?.15 (OUT10): now also D?.1 (K)
- net at U?.16 (OUT11): now also D?.1 (K)
- net at U?.23 (SET): now also R?.1
- net at U?.5 (OUT0): now also D?.1 (K)
- net at U?.6 (OUT1): now also D?.1 (K)
- net at U?.8 (OUT3): now also D?.1 (K)
- net at U?.9 (OUT4): now also D?.1 (K)
- no-connect marks 5 -> 10

Commit message: Commit from work, almost done with layout.
Parts:
- removed SW?: SW_Push_HeadingSync, symbol Switch:SW_Push
- added R? (x8): 10k Ohm, symbol Device:R
- added SW?: RotaryEncoder_Alt1000, symbol Device:RotaryEncoder
- added SW?: RotaryEncoder_HeadingSelect, symbol Device:RotaryEncoder_Switch
- added SW?: RotaryEncoder_VSSelect, symbol Device:RotaryEncoder
- added SW?: RotaryEncoder_Alt100, symbol Device:RotaryEncoder
Connections:
- net GND: now also SW?.C, SW?.C, SW?.C, SW?.C
- net VCC: now also R?.2, R?.2, R?.2, R?.2, R?.2, R?.2, R?.2, R?.2, SW?.S1; no longer J?.1 (VBUS), U?.18 (VUSB)
- net Heading_Sync: now reaches U?.1 (I3)
- net Heading_Sync: now also SW?.S2
- net at U?.19 (SPP0/RD0): now also R?.1, SW?.A
- net at U?.20 (SPP1/RD1): now also R?.1, SW?.B
- net at U?.21 (SPP2/RD2): now also R?.1, SW?.A
- net at U?.22 (SPP3/RD3): now also R?.1, SW?.B
- net at U?.27 (SPP4/RD4): now also R?.1, SW?.A
- net at U?.28 (P1B/SPP5/RD5): now also R?.1, SW?.B
- net at U?.29 (P1C/SPP6/RD6): now also R?.1, SW?.A
- net at U?.30 (P1D/SPP7/RD7): now also R?.1, SW?.B
- new net VBUS: J?.1 (VBUS)
Other:
- moved on the sheet: J?
